File: prj/extUsb/extUsb.kicad_pcb (KiCad board)
At the start: 2 copper layers, 21.7 x 12.7 mm, 20 parts, among them J1 USB_B_Micro, J2 Conn_01x05, U1 SN74LVC2T45, U2 MIC5504-3.3YM5, U3 TS5A3166DBVR

Commit message: extUsb Final release suitable for laser-etch or commercial fabs.
Routing:
- net pin_usb_oe: track 18.4 -> 20.0 mm
